Commit message: fix: now right should is aligned with actual robot

File: urdf/R1Mk3/robots/R1SN003/model.urdf (robot description, URDF)
Before this commit: robot R1Mk3, 182 links, 181 joints
Links:
- removed link mobile_base_lidar
- added link mobile_base_double_lidar
Joints:
- removed joint mobile_base_lidar_fixed_joint
- added joint mobile_base_double_lidar_fixed_joint: type fixed, parent mobile_base_body_link, child mobile_base_double_lidar, origin xyz=0.0 0 0.031 rpy=0 -0 0
- joint depth_center_fixed_joint: origin xyz=0.05132104198001797 5.593391840255621e-17 0.05375374559540269 rpy=-1.3962634015954642 -1.0632884247878182e-17 -1.5707963267948954 -> xyz=0.05132104198001797 5.593391840255621e-17 0.05375374559540269 rpy=-1.57079 -1.0632884247878182e-17 -1.5707963267948954
- joint neck_pitch_joint: axis -1.1561757607518887e-15 -1 5.551115123110952e-17 -> -1.1561757607518887e-15 1 5.551115123110952e-17; origin xyz=-0.0939999999999997 -1.5911115898279495e-16 0.3304999999999986 rpy=1.4266365866433113e-14 1.1313955190051007e-15 4.4868448346273745e-15 -> xyz=-0.0939999999999997 -1.5911115898279495e-16 0.33 rpy=1.4266365866433113e-14 1.1313955190051007e-15 4.4868448346273745e-15
- joint neck_yaw_joint: axis -5.551115123125783e-17 1.0407701698506794e-17 -1.0000000000000002 -> 0.0 1.0407701698506794e-17 -1.0; origin xyz=0.011679488023179689 -9.677503327256982e-18 0.1583779958185998 rpy=-1.2299256863622814e-15 0.17453292519943311 -7.040232933848852e-15 -> xyz=0.011679488023179689 -9.677503327256982e-18 0.1583779958185998 rpy=-1.2299256863622814e-15 0.17 -7.040232933848852e-15
- joint r_shoulder_roll: origin xyz=0.003749999999999143 -0.09330000000000055 -0.006495190528383377 rpy=0.244346095279198 1.0471975511965996 2.4338251683117622e-14 -> xyz=0.003749999999999143 -0.09330000000000055 -0.006495190528383377 rpy=0.0 1.0471975511965996 2.4338251683117622e-14
- joint torso_pitch_eq_joint: origin xyz=-1.3183898417423734e-16 -5.769801341748891e-19 -8.881784197001252e-16 rpy=2.677430187438326e-32 1.110223024625156e-16 -1.2767564783189298e-15 -> xyz=-1.3183898417423734e-16 -5.769801341748891e-19 -8.881784197001252e-16 rpy=0.0 1.110223024625156e-16 -1.2767564783189298e-15
- joint torso_roll_eq_joint: origin xyz=2.0816681711721685e-17 -5.242619982186716e-24 0.40000000000000024 rpy=0 2.220446049250313e-16 -1.8377532023260753e-23 -> xyz=2.0816681711721685e-17 -5.242619982186716e-24 0.40000000000000024 rpy=0.0 0.0 -1.8377532023260753e-23
- joint torso_yaw_joint: axis 1.4574786319396409e-16 1.0898835157993226e-15 -1 -> 1.4574786319396409e-16 1.0898835157993226e-15 1; origin xyz=2.220446049250313e-16 -1.6880686544087094e-16 0.06950000000000012 rpy=-1.0898835157993226e-15 1.4574786319396409e-16 2.150984683485474e-15 -> xyz=2.220446049250313e-16 -1.6880686544087094e-16 0.07 rpy=-1.0898835157993226e-15 1.4574786319396409e-16 2.150984683485474e-15
